File: Electron/V1/PCB/WaterMonitor.brd (EAGLE design)
At the start: 95.9 x 34.6 mm, 36 parts, among them U1 SN74LV8154PW, U2 ELECTRONDUALNAMED, U3 24LC512

Commit message: Minor tidy for part names etc.
Added pdf's for V1 PCB.
Parts:
- R1: value (none) -> 1k
- renumbered U$1 to U4

Commit message: V1.1 changes - not sure what. Not important - not using this version any more.
Parts:
- removed C4: 0.1uF, SparkFun-Passives:0805
- removed JP4: ColdFlow, SparkFun-Connectors:MOLEX-1X3
- removed JP5: HotFlow, SparkFun-Connectors:MOLEX-1X3
- removed U3: 24LC512, SparkFun-DigitalIC:SO08
- added J1, J2: (no value), Tinamous:JST-HX-3-PTH-VERT
- R2: value 10k -> 4k7
- R3, R4: value 2k -> 100R
- moved R4 25.2 mm to (91.4, 9.53), turned to 0 degrees
- moved R3 20.4 mm to (92.7, 19.1), turned to 270 degrees
- moved U4 14.7 mm to (67.0, 12.7), turned to 0 degrees
- moved R12 9.55 mm to (29.2, 7.62)
- moved C5 8.89 mm to (64.8, 6.99), turned to 0 degrees
- moved R2 3.13 mm to (89.5, 2.22)
- moved C6 1.59 mm to (105.7, 16.8), turned to 180 degrees
- moved R5 0.64 mm to (40.0, -2.54)
- moved R6 0.64 mm to (45.7, -2.54)
- moved R7 0.64 mm to (34.3, -2.54)
- moved R8 0.64 mm to (50.8, -2.54)
- moved C3 0.63 mm to (24.4, -2.22)
- turned C1 to 270 degrees
Connections:
- new net N$3: J1.3, R3.1
- new net N$4: J2.3, R4.2
- net 3.3V: now also R5.1, R6.1, R7.1, R8.1; no longer C4.2, R3.2, R4.2, U3.8
- net 5V: now also J1.1, J2.1; no longer JP4.3, JP5.3
- net COLD_FLOW: now also R3.2; no longer JP4.2
- net GND: now also J1.2, J2.2; no longer C4.1, JP4.1, JP5.1, R5.1, R6.1, R7.1, R8.1, U3.1, U3.2, U3.3, U3.4, U3.7
- net HOT_FLOW: now also R4.1; no longer JP5.2
- net SCL: no longer R4.1, U3.6
- net SDA: no longer R3.1, U3.5
Routing:
- net SCL: track 41.3 -> 2.54 mm, vias 2 -> 0
- net SDA: track 35.8 -> 2.54 mm
- net 3.3V: track 188.1 -> 210.4 mm
- net N$4: track 0.00 -> 13.2 mm
- net HOT_FLOW: track 65.8 -> 53.5 mm, vias 2 -> 3
- net COLD_FLOW: track 75.4 -> 67.4 mm
- net N$3: track 0.00 -> 6.68 mm
- net DQ: track 89.8 -> 94.1 mm
- net GND: track 9.11 -> 6.57 mm, vias 5 -> 7
- net 5V: track 138.7 -> 140.3 mm
- net OSH_LOGO_LED: track 92.1 -> 93.0 mm
- net HOT_LOW_BYTE: track 10.7 -> 11.4 mm
- net HOT_HIGH_BYTE: track 13.1 -> 13.7 mm
- net COLD_LOW_BYTE: track 14.3 -> 14.9 mm
- net COLD_HIGH_BYTE: track 11.2 -> 11.8 mm
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Other:
- board text added: "3v3"
- board text added: "5V"
- board text added: "DQ"
- board text added: "FLOW"
- board text added: "GND"
- board text added: "Pulse"
- board text added: "Temperature"
- board text added: "V1.1"
- board text removed: "DS18B20"
- board text removed: "FLOW (5V)"
- board text removed: "FLOW(5V)"
- board text removed: "V1.00"
