File: Electron/V1/PCB/WaterMonitor.sch (EAGLE design)
At the start: 36 parts, among them U1 SN74LV8154PW, U2 ELECTRONDUALNAMED, U3 24LC512

Commit message: Minor tidy for part names etc.
Added pdf's for V1 PCB.
Parts:
- R1: value (none) -> 1k
- renumbered U$1 to U4
Other:
- moved on the sheet: H1, H2, H3
Changed lines of the file:
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@@
 <part name="LOGO1" library="SparkFun-Aesthetics" deviceset="OSHW-LOGO" device="M"/>
 <part name="D1" library="SparkFun-LED" deviceset="LED" device="1206-BOTTOM"/>
-<part name="R1" library="SparkFun-Resistors" deviceset="RESISTOR" device="1206"/>
+<part name="R1" library="SparkFun-Resistors" deviceset="RESISTOR" device="1206" value="1k"/>
 <part name="GND4" library="SparkFun-Aesthetics" deviceset="DGND" device=""/>
 <part name="U3" library="SparkFun-DigitalIC" deviceset="EEPROM-I2C" device="SMD" value="24LC512">
@@
 <part name="SUPPLY3" library="SparkFun-Aesthetics" deviceset="3.3V" device=""/>
 <part name="GND6" library="SparkFun-Aesthetics" deviceset="DGND" device=""/>
-<part name="U$1" library="DS1820-SOIC" deviceset="DS1820" device="SOIC"/>
+<part name="U4" library="DS1820-SOIC" deviceset="DS1820" device="SOIC"/>
 <part name="GND7" library="SparkFun-Aesthetics" deviceset="DGND" device=""/>
 <part name="SUPPLY5" library="SparkFun-Aesthetics" deviceset="3.3V" device=""/>
@@
 <text x="190.5" y="167.64" size="1.27" layer="97">Battery</text>
 <text x="243.84" y="114.3" size="1.27" layer="97">Cold Temperature Sensor</text>
+<wire x1="180.34" y1="187.96" x2="271.78" y2="187.96" width="0.1524" layer="97"/>
+<wire x1="271.78" y1="124.46" x2="271.78" y2="187.96" width="0.1524" layer="97"/>
+<wire x1="180.34" y1="124.46" x2="180.34" y2="187.96" width="0.1524" layer="97"/>
+<wire x1="271.78" y1="124.46" x2="180.34" y2="124.46" width="0.1524" layer="97"/>
 </plain>
 <instances>
@@
 <instance part="SUPPLY2" gate="G$1" x="104.14" y="152.4"/>
 <instance part="GND2" gate="G$1" x="83.82" y="147.32" rot="R270"/>
-<instance part="H1" gate="G$1" x="251.46" y="180.34"/>
-<instance part="H2" gate="G$1" x="251.46" y="172.72"/>
+<instance part="H1" gate="G$1" x="243.84" y="180.34"/>
+<instance part="H2" gate="G$1" x="243.84" y="172.72"/>
 <instance part="SUPPLY4" gate="G$1" x="134.62" y="152.4"/>
 <instance part="U2" gate="G$1" x="116.84" y="129.54"/>
@@
 <instance part="SUPPLY3" gate="G$1" x="157.48" y="38.1"/>
 <instance part="GND6" gate="G$1" x="157.48" y="25.4"/>
-<instance part="U$1" gate="G$1" x="208.28" y="58.42"/>
+<instance part="U4" gate="G$1" x="208.28" y="58.42"/>
 <instance part="GND7" gate="G$1" x="205.74" y="43.18"/>
 <instance part="SUPPLY5" gate="G$1" x="220.98" y="66.04"/>
@@
 <instance part="GND14" gate="G$1" x="203.2" y="154.94"/>
 <instance part="SUPPLY14" gate="G$1" x="210.82" y="165.1"/>
-<instance part="H3" gate="G$1" x="251.46" y="165.1"/>
+<instance part="H3" gate="G$1" x="243.84" y="165.1"/>
 <instance part="D3" gate="G$1" x="205.74" y="162.56"/>
 <instance part="R2" gate="G$1" x="228.6" y="53.34" rot="R90"/>
@@
 </segment>
 <segment>
-<pinref part="U$1" gate="G$1" pin="GND"/>
+<pinref part="U4" gate="G$1" pin="GND"/>
 <pinref part="GND7" gate="G$1" pin="GND"/>
 <wire x1="205.74" y1="53.34" x2="205.74" y2="45.72" width="0.1524" layer="91"/>
@@
 </segment>
 <segment>
-<pinref part="U$1" gate="G$1" pin="VCC"/>
+<pinref part="U4" gate="G$1" pin="VCC"/>
 <wire x1="210.82" y1="53.34" x2="210.82" y2="48.26" width="0.1524" layer="91"/>
 <pinref part="SUPPLY5" gate="G$1" pin="3.3V"/>
@@
 <net name="DQ" class="0">
 <segment>
-<pinref part="U$1" gate="G$1" pin="DQ"/>
+<pinref part="U4" gate="G$1" pin="DQ"/>
 <wire x1="208.28" y1="53.34" x2="208.28" y2="45.72" width="0.1524" layer="91"/>
 <wire x1="208.28" y1="45.72" x2="228.6" y2="45.72" width="0.1524" layer="91"/>

Commit message: Tidy up
Other:
- note added: "NB: Should these be pulled high as they are active low."
- moved on the sheet: C1, C2, C3, C4, C5, C6, CONN1, D1, D2, D3, H1, H2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

Commit message: V1.1 changes - not sure what. Not important - not using this version any more.
Parts:
- removed C4: 0.1uF, SparkFun-Passives:CAP0805
- removed JP4: ColdFlow, SparkFun-Connectors:M03POLAR
- removed JP5: HotFlow, SparkFun-Connectors:M03POLAR
- removed U3: 24LC512, SparkFun-DigitalIC:EEPROM-I2CSMD
- added J1, J2: (no value), Tinamous:CONN_03JST-HX-PTH-VERT
- R2: value 10k -> 4k7
- R3, R4: value 2k -> 100R
Connections:
- new net N$3: J1.3, R3.1
- new net N$4: J2.3, R4.2
- net 3.3V: now also R5.1, R6.1, R7.1, R8.1; no longer C4.2, R3.2, R4.2, U3.VCC
- net 5V: now also J1.1, J2.1; no longer JP4.3, JP5.3
- net COLD_FLOW: now also R3.2; no longer JP4.2
- net GND: now also J1.2, J2.2; no longer C4.1, JP4.1, JP5.1, R5.1, R6.1, R7.1, R8.1, U3.A0, U3.A1, U3.A2, U3.VSS, U3.WP
- net HOT_FLOW: now also R4.1; no longer JP5.2
- net SCL: no longer R4.1, U3.SCL
- net SDA: no longer R3.1, U3.SDA
Other:
- note removed: "1010 000r xxxx xxxx xxxx xxxx r=read/write operation 1 = read 0=write"
- note removed: "Address: Control: A0 + Address High + Address Low"
- note removed: "Data Logging"
- moved on the sheet: C1, C6, D3, H1, H2, H3, JP1, JP2, JP3, R10, R3, R4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
