File: Electron/V2/PCB/WaterMonitorV2.1.brd (EAGLE design)
At the start: 100 x 50 mm, 57 parts, among them IC1 7805DT, J1 ColdFlow, J2 HotFlow, J3 Cold Valve, J4 Hot Valve, J6 POWER_JACKPTH_LOCK, J9 JST PH - Grove, Q1 4.3A/20V/54mΩ, Q3 220mA/50V/3.5Ω, Q5 4.3A/20V/54mΩ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

Commit message: Added images for V2.1
Remove todo text from schematic.

Changed water sense fault net to water sense power.
Connections:
- net WATER_SENSE_FAULT renamed WATER_SENSE_POWER
Changed lines of the file:
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@@
 <wire x1="33.9725" y1="-4.7625" x2="33.9725" y2="2.2225" width="0.4064" layer="1"/>
 </signal>
-<signal name="WATER_SENSE_FAULT">
+<signal name="WATER_SENSE_POWER">
 <contactref element="JP3" pad="4"/>
 <contactref element="MS1" pad="#7"/>
