File: Electron/V2/PCB/WaterMonitorV2.1.sch (EAGLE design)
At the start: 57 parts, among them IC1 7805DT, J1 ColdFlow, J2 HotFlow, J3 Cold Valve, J4 Hot Valve, J6 POWER_JACKPTH_LOCK, J9 JST PH - Grove, Q1 4.3A/20V/54mΩ, Q3 220mA/50V/3.5Ω, Q5 4.3A/20V/54mΩ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

Commit message: Added images for V2.1
Remove todo text from schematic.

Changed water sense fault net to water sense power.
Connections:
- net WATER_SENSE_FAULT renamed WATER_SENSE_POWER
Other:
- note removed: "TODO: * Room temperature (and humidity?) * Don't use D13 for OSH Logo LED as its's also onboard LED. * Add buzzer? LED? for leak * Bigger holes needed for 3 pin JST"
- note removed: "TODO: Need power to sensor board. - Use fault to provide power."
- note removed: "WATER_SENSE_FAULT - should connect to GND in the external sensor."
Changed lines of the file:
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@@
 <wire x1="2.54" y1="129.54" x2="2.54" y2="73.66" width="0.1524" layer="97"/>
 <text x="78.74" y="185.42" size="1.27" layer="97">Water leak sensor.</text>
-<text x="78.74" y="134.62" size="1.27" layer="97">WATER_SENSE_FAULT - should connect to GND in the external sensor.</text>
 <text x="78.74" y="139.7" size="1.27" layer="97">WATER_SENSE_1 and 2 - should connect to GND in the external sensor when water is present.</text>
-<text x="81.28" y="287.02" size="1.27" layer="97">TODO:
-* Room temperature (and humidity?)
-* Don't use D13 for OSH Logo LED as its's also onboard LED.
-* Add buzzer? LED? for leak
-* Bigger holes needed for 3 pin JST
-</text>
-<text x="78.74" y="149.86" size="1.27" layer="97">TODO: Need power to sensor board. - Use fault to provide power.</text>
 <text x="15.24" y="264.16" size="1.27" layer="97">TODO: Check SDA/SCL ok with 5V display</text>
 <wire x1="193.04" y1="149.86" x2="426.72" y2="149.86" width="0.1524" layer="97"/>
@@
 </segment>
 </net>
-<net name="WATER_SENSE_FAULT" class="0">
+<net name="WATER_SENSE_POWER" class="0">
 <segment>
 <pinref part="JP3" gate="G$1" pin="4"/>
