File: Feather/V7/PCB/WaterMonitorV7.0.sch (EAGLE design)
At the start: 45 parts, among them IC1 BME680, J3 Flow1, J4 Flow2, J6 Temperature2, J7 Temperature1, Q1 4.3A/20V/54mΩ, Q3 220mA/50V/3.5Ω

Commit message: Moved OSH LED, added values.
Parts:
- J3, J4: FARNELL (none) -> 1516227
- Q1: value 4.3A/20V/54mΩ -> IRLML2244TRPBF; FARNELL (none) -> 2468051
- Q3: value 220mA/50V/3.5Ω -> BSS138PW; FARNELL (none) -> 1907611
Connections:
- net FLOW_1: now also MS1.GPIO5; no longer MS1.GPIO6
- net FLOW_2: now also MS1.GPIO6; no longer MS1.GPIO5
- net FLOW_3: now also MS1.GPIO10; no longer MS1.GPIO11
- net FLOW_4: now also MS1.GPIO11; no longer MS1.GPIO10
- net OSH_LOGO_LED: now also MS1.GPIOTX; no longer MS1.GPIOMOSI
Changed lines of the file:
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@@
 <part name="FRAME2" library="SparkFun-Aesthetics" deviceset="FRAME-LEDGER" device=""/>
 <part name="R4" library="SparkFun-Resistors" deviceset="RESISTOR" device="0805" value="1k"/>
-<part name="Q1" library="SparkFun-DiscreteSemi" deviceset="MOSFET_PCH" device="-IRLML2244" value="4.3A/20V/54mΩ"/>
+<part name="Q1" library="SparkFun-DiscreteSemi" deviceset="MOSFET_PCH" device="-IRLML2244" value="IRLML2244TRPBF">
+<attribute name="FARNELL" value="2468051"/>
+</part>
 <part name="SUPPLY10" library="SparkFun-Aesthetics" deviceset="5V" device=""/>
 <part name="R15" library="SparkFun-Resistors" deviceset="RESISTOR" device="0805" value="1M"/>
-<part name="Q3" library="SparkFun-DiscreteSemi" deviceset="MOSFET-NCH" device="-BSS138" value="220mA/50V/3.5Ω"/>
+<part name="Q3" library="SparkFun-DiscreteSemi" deviceset="MOSFET-NCH" device="-BSS138" value="BSS138PW">
+<attribute name="FARNELL" value="1907611"/>
+</part>
 <part name="GND19" library="SparkFun-Aesthetics" deviceset="DGND" device=""/>
 <part name="R5" library="SparkFun-Resistors" deviceset="RESISTOR" device="0805" value="1M"/>
@@
 <part name="R7" library="SparkFun-Resistors" deviceset="RESISTOR" device="0805" value="100k"/>
 <part name="GND12" library="SparkFun-Aesthetics" deviceset="DGND" device=""/>
-<part name="J3" library="Tinamous" deviceset="CONN_03" device="JST-HX-PTH-VERT" value="Flow1"/>
+<part name="J3" library="Tinamous" deviceset="CONN_03" device="JST-HX-PTH-VERT" value="Flow1">
+<attribute name="FARNELL" value="1516227"/>
+</part>
 <part name="R12" library="SparkFun-Resistors" deviceset="RESISTOR" device="0805" value="1k"/>
 <part name="GND13" library="SparkFun-Aesthetics" deviceset="DGND" device=""/>
 <part name="R13" library="SparkFun-Resistors" deviceset="RESISTOR" device="0805" value="100k"/>
 <part name="GND16" library="SparkFun-Aesthetics" deviceset="DGND" device=""/>
-<part name="J4" library="Tinamous" deviceset="CONN_03" device="JST-HX-PTH-VERT" value="Flow2"/>
+<part name="J4" library="Tinamous" deviceset="CONN_03" device="JST-HX-PTH-VERT" value="Flow2">
+<attribute name="FARNELL" value="1516227"/>
+</part>
 <part name="R14" library="SparkFun-Resistors" deviceset="RESISTOR" device="0805" value="1k"/>
 <part name="GND17" library="SparkFun-Aesthetics" deviceset="DGND" device=""/>
@@
 <attribute name="VALUE" x="24.13" y="50.038" size="1.778" layer="96"/>
 </instance>
-<instance part="Q1" gate="G$1" x="363.22" y="246.38" rot="R180"/>
+<instance part="Q1" gate="G$1" x="363.22" y="246.38" rot="R180">
+<attribute name="FARNELL" x="363.22" y="246.38" size="1.778" layer="96" rot="R180" display="off"/>
+</instance>
 <instance part="SUPPLY10" gate="G$1" x="360.68" y="266.7"/>
 <instance part="R15" gate="G$1" x="370.84" y="256.54" smashed="yes" rot="R90">
@@
 <attribute name="VALUE" x="374.142" y="255.27" size="1.778" layer="96" rot="R90"/>
 </instance>
-<instance part="Q3" gate="NMOS" x="381" y="243.84" rot="MR0"/>
+<instance part="Q3" gate="NMOS" x="381" y="243.84" rot="MR0">
+<attribute name="FARNELL" x="381" y="243.84" size="1.778" layer="96" rot="MR0" display="off"/>
+</instance>
 <instance part="GND19" gate="G$1" x="378.46" y="228.6"/>
 <instance part="R5" gate="G$1" x="388.62" y="233.68" smashed="yes" rot="R180">
@@
 <attribute name="VALUE" x="227.076" y="247.142" size="1.778" layer="96" font="vector"/>
 <attribute name="NAME" x="233.68" y="235.712" size="1.778" layer="95" font="vector" rot="R180"/>
+<attribute name="FARNELL" x="231.14" y="241.3" size="1.778" layer="96" rot="R180" display="off"/>
 </instance>
 <instance part="R12" gate="G$1" x="213.36" y="238.76" smashed="yes">
@@
 <attribute name="VALUE" x="282.956" y="247.142" size="1.778" layer="96" font="vector"/>
 <attribute name="NAME" x="289.56" y="235.712" size="1.778" layer="95" font="vector" rot="R180"/>
+<attribute name="FARNELL" x="287.02" y="241.3" size="1.778" layer="96" rot="R180" display="off"/>
 </instance>
 <instance part="R14" gate="G$1" x="269.24" y="238.76" smashed="yes">
@@
 </segment>
 <segment>
-<pinref part="MS1" gate="G$1" pin="GPIOMOSI"/>
-<wire x1="104.14" y1="223.52" x2="99.06" y2="223.52" width="0.1524" layer="91"/>
-<label x="99.06" y="223.52" size="1.27" layer="95" rot="R180" xref="yes"/>
+<pinref part="MS1" gate="G$1" pin="GPIOTX"/>
+<wire x1="104.14" y1="215.9" x2="99.06" y2="215.9" width="0.1524" layer="91"/>
+<label x="99.06" y="215.9" size="1.27" layer="95" rot="R180" xref="yes"/>
 </segment>
 </net>
@@
 </segment>
 <segment>
-<pinref part="MS1" gate="G$1" pin="GPIO11"/>
-<wire x1="147.32" y1="228.6" x2="152.4" y2="228.6" width="0.1524" layer="91"/>
-<label x="152.4" y="228.6" size="1.27" layer="95" xref="yes"/>
+<pinref part="MS1" gate="G$1" pin="GPIO10"/>
+<wire x1="147.32" y1="226.06" x2="152.4" y2="226.06" width="0.1524" layer="91"/>
+<label x="152.4" y="226.06" size="1.27" layer="95" xref="yes"/>
 </segment>
 </net>
@@
 </segment>
 <segment>
-<pinref part="MS1" gate="G$1" pin="GPIO6"/>
-<wire x1="147.32" y1="220.98" x2="152.4" y2="220.98" width="0.1524" layer="91"/>
-<label x="152.4" y="220.98" size="1.27" layer="95" xref="yes"/>
+<pinref part="MS1" gate="G$1" pin="GPIO5"/>
+<wire x1="147.32" y1="218.44" x2="152.4" y2="218.44" width="0.1524" layer="91"/>
+<label x="152.4" y="218.44" size="1.27" layer="95" xref="yes"/>
 </segment>
 </net>
@@
 </segment>
 <segment>
-<pinref part="MS1" gate="G$1" pin="GPIO5"/>
-<wire x1="147.32" y1="218.44" x2="152.4" y2="218.44" width="0.1524" layer="91"/>
-<label x="152.4" y="218.44" size="1.27" layer="95" xref="yes"/>
+<pinref part="MS1" gate="G$1" pin="GPIO6"/>
+<wire x1="147.32" y1="220.98" x2="152.4" y2="220.98" width="0.1524" layer="91"/>
+<label x="152.4" y="220.98" size="1.27" layer="95" xref="yes"/>
 </segment>
 </net>
@@
 </segment>
 <segment>
-<pinref part="MS1" gate="G$1" pin="GPIO10"/>
-<wire x1="147.32" y1="226.06" x2="152.4" y2="226.06" width="0.1524" layer="91"/>
-<label x="152.4" y="226.06" size="1.27" layer="95" xref="yes"/>
-</segment>
-</net>
+<pinref part="MS1" gate="G$1" pin="GPIO11"/>
+<wire x1="147.32" y1="228.6" x2="152.4" y2="228.6" width="0.1524" layer="91"/>
+<label x="152.4" y="228.6" size="1.27" layer="95" xref="yes"/>
+</segment>
+</net>
